File: CarrierBoard_CmodA7/CarrierBoard_CmodA7.kicad_sch (KiCad schematic)
At the start: 67 parts, among them CN1 Mini-Fit_Jr._Header,_2_Circui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, J1 Conn1x22, J2 Conn1x27, U1 AZ1084CD-5.0, U2 Cmod_A7, U3 PMOD_GPIO, U4 PMOD_GPIO, U5 PMOD_GPIO, U6 PMOD_GPIO

Commit message: Arreglado BoM y esquemas
Parts:
- C1, C3: value Gen_C -> 10uF
- C2, C4: value Gen_C -> 100nF
- C5, C6: value Gen_C -> 1nF
Changed lines of the file:
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@@
   (symbol (lib_id "Herranz - Capacitor (0603):Gen_C") (at 182 39 0) (unit 1)
     (in_bom yes) (on_board yes) (fields_autoplaced)
-    (property "Reference" "C6" (id 0) (at 186.06 43.7299 0)
-      (effects (font (size 1.27 1.27)) (justify left))
-    )
-    (property "Value" "Gen_C" (id 1) (at 186.06 46.2699 0)
+    (property "Reference" "C6" (id 0) (at 185.42 43.7299 0)
+      (effects (font (size 1.27 1.27)) (justify left))
+    )
+    (property "Value" "1nF" (id 1) (at 185.42 46.2699 0)
       (effects (font (size 1.27 1.27)) (justify left))
     )
@@
   (symbol (lib_id "Herranz - Capacitor (0805):Gen_C") (at 37 38 0) (unit 1)
     (in_bom yes) (on_board yes) (fields_autoplaced)
-    (property "Reference" "C1" (id 0) (at 41.13 40.7699 0)
-      (effects (font (size 1.27 1.27)) (justify left))
-    )
-    (property "Value" "Gen_C" (id 1) (at 41.13 43.3099 0)
+    (property "Reference" "C1" (id 0) (at 40.64 40.7699 0)
+      (effects (font (size 1.27 1.27)) (justify left))
+    )
+    (property "Value" "10uF" (id 1) (at 40.64 43.3099 0)
       (effects (font (size 1.27 1.27)) (justify left))
     )
@@
   (symbol (lib_id "Herranz - Capacitor (0805):Gen_C") (at 85 38 0) (unit 1)
     (in_bom yes) (on_board yes) (fields_autoplaced)
-    (property "Reference" "C4" (id 0) (at 88.66 40.7699 0)
-      (effects (font (size 1.27 1.27)) (justify left))
-    )
-    (property "Value" "Gen_C" (id 1) (at 88.66 43.3099 0)
+    (property "Reference" "C4" (id 0) (at 88.9 40.7699 0)
+      (effects (font (size 1.27 1.27)) (justify left))
+    )
+    (property "Value" "100nF" (id 1) (at 88.9 43.3099 0)
       (effects (font (size 1.27 1.27)) (justify left))
     )
@@
       (effects (font (size 1.27 1.27)) (justify left))
     )
-    (property "Value" "Gen_C" (id 1) (at 76.2 43.3099 0)
+    (property "Value" "10uF" (id 1) (at 76.2 43.3099 0)
       (effects (font (size 1.27 1.27)) (justify left))
     )
@@
   (symbol (lib_id "Herranz - Capacitor (0603):Gen_C") (at 132 39 0) (unit 1)
     (in_bom yes) (on_board yes) (fields_autoplaced)
-    (property "Reference" "C5" (id 0) (at 135.1 43.7299 0)
-      (effects (font (size 1.27 1.27)) (justify left))
-    )
-    (property "Value" "Gen_C" (id 1) (at 135.1 46.2699 0)
+    (property "Reference" "C5" (id 0) (at 135.89 43.7299 0)
+      (effects (font (size 1.27 1.27)) (justify left))
+    )
+    (property "Value" "1nF" (id 1) (at 135.89 46.2699 0)
       (effects (font (size 1.27 1.27)) (justify left))
     )
@@
       (effects (font (size 1.27 1.27)) (justify left))
     )
-    (property "Value" "Gen_C" (id 1) (at 52.07 43.3099 0)
+    (property "Value" "100nF" (id 1) (at 52.07 43.3099 0)
       (effects (font (size 1.27 1.27)) (justify left))
     )
@@
     )
     (path "/62efff76-31b2-4532-92f3-a119f6b7126c"
-      (reference "C1") (unit 1) (value "Gen_C") (footprint "Capacitor_SMD:C_0805_2012Metric")
+      (reference "C1") (unit 1) (value "10uF") (footprint "Capacitor_SMD:C_0805_2012Metric")
     )
     (path "/c4524e0f-4ff7-4488-b8a2-8cc0fb12622d"
-      (reference "C2") (unit 1) (value "Gen_C") (footprint "Capacitor_SMD:C_0805_2012Metric")
+      (reference "C2") (unit 1) (value "100nF") (footprint "Capacitor_SMD:C_0805_2012Metric")
     )
     (path "/a80f005d-9e50-4166-a1a5-61f760546419"
-      (reference "C3") (unit 1) (value "Gen_C") (footprint "Capacitor_SMD:C_0805_2012Metric")
+      (reference "C3") (unit 1) (value "10uF") (footprint "Capacitor_SMD:C_0805_2012Metric")
     )
     (path "/63cf5d7e-9450-42b5-a059-62cb491ffe1e"
-      (reference "C4") (unit 1) (value "Gen_C") (footprint "Capacitor_SMD:C_0805_2012Metric")
+      (reference "C4") (unit 1) (value "100nF") (footprint "Capacitor_SMD:C_0805_2012Metric")
     )
     (path "/be6931f5-6deb-45f1-a513-96b0a11abc02"
-      (reference "C5") (unit 1) (value "Gen_C") (footprint "Capacitor_SMD:C_0603_1608Metric")
+      (reference "C5") (unit 1) (value "1nF") (footprint "Capacitor_SMD:C_0603_1608Metric")
     )
     (path "/5f372e0b-ba88-473c-8f10-21d735427607"
-      (reference "C6") (unit 1) (value "Gen_C") (footprint "Capacitor_SMD:C_0603_1608Metric")
+      (reference "C6") (unit 1) (value "1nF") (footprint "Capacitor_SMD:C_0603_1608Metric")
     )
     (path "/88f84aee-48ca-49a2-8c37-f5c5ee5ca717"
